Commit message: Updated robotiq with untracked changes for APC

File: robotiq_s_model_visualization/cfg_NEW/s-model_articulated_macro.xacro (robot description, xacro)
@@ -23,5 +23,5 @@
 			<collision>
 				<geometry>
-					<mesh filename="package://robotiq_s_model_visualization/meshes/s-model_articulated/visual/palm.STL" />
+					<mesh filename="package://robotiq_s_model_visualization/meshes/s-model_articulated/collision/palm.STL" />
 				</geometry>
 				<material name="yellow">
@@ -34,4 +34,30 @@
             <mass value="1.3"/>
             <inertia ixx="0.006012" ixy="0.000079" ixz="-0.00024" iyy="0.012892" iyz="0" izz="0.002435" />
+        </inertial>
+        <!-- Collision Sphere Test-->
+		<link name="${prefix}collision_sphere_joint">
+			<visual>
+				<geometry>
+					<!--<mesh filename="package://robotiq_s_model_visualization/meshes/s-model_articulated/visual/ball.stl" />-->
+                    <sphere radius = "0.1"/>
+				</geometry>
+				<material name="green">
+					<color rgba="0 1 0 1"/>
+				</material>
+			</visual>
+			<collision>
+				<geometry>
+					<!-- <mesh filename="package://robotiq_s_model_visualization/meshes/s-model_articulated/collision/ball.stl" /> -->
+                    <sphere radius = "0.1"/>
+				</geometry>
+				<material name="red">
+					<color rgba="1 0 0 1"/>
+				</material>
+			</collision>
+		</link>
+        <inertial>
+            <origin xyz="0 0 0" rpy="0 0 0"/>
+            <mass value="1.0"/>
+            <inertia ixx="0" ixy="0" ixz="0" iyy="0" iyz="0" izz="0" />
         </inertial>
 		<!-- end of link list -->
@@ -61,7 +87,3 @@
 		<!-- end of joint list -->
 	</xacro:macro>
-<gazebo>
-  <plugin name="RobotiqHandPlugin" filename="libRobotiqHandPlugin.so">
-  </plugin>
-</gazebo>
 </robot>

File: robotiq_s_model_visualization/cfg_NEW/s-model_finger_articulated_macro.xacro (robot description, xacro)
@@ -19,6 +19,5 @@
 			</visual>
 			<collision>
-				<!--<origin xyz="-0.0455 0.0414 0.036" rpy="0 3.1416 -1.57"/>-->
-                <origin xyz="0.020 0 0" rpy="0 0 0"/>
+				<origin xyz="-0.0455 0.0414 0.036" rpy="0 3.1416 -1.57"/>
 				<geometry>
 					<mesh filename="package://robotiq_s_model_visualization/meshes/s-model_articulated/collision/link_0.STL" />
