Commit message: Added real finger extensions

File: robotiq_s_model_visualization/cfg/s-model_finger_articulated_macro.xacro (robot description, xacro)
@@ -82,16 +82,18 @@
 		<link name="${prefix}link_3">
 			<visual>
-				<origin xyz="0.075 0.03 0" rpy="0 0 0.52"/>
+				<origin xyz="0 -0.0025 0.015" rpy="1.57079632679 1.57079632679 0.52"/>
 				<geometry>
 					<!-- <mesh filename="package://robotiq_s_model_visualization/meshes/s-model_articulated/visual/link_3.STL" /> -->
-					<box size="0.15 0.03 0.03" />
+					<mesh filename="package://robotiq_s_model_visualization/meshes/s-model_articulated/visual/extensions.STL" />
+					<!-- <box size="0.15 0.03 0.03" /> -->
 				</geometry>
 				<material name="green"/>
 			</visual>
 			<collision>
-				<origin xyz="0.075 0.03 0" rpy="0 0 0.52"/>
+				<origin xyz="0 -0.0025 0.015" rpy="1.57079632679 1.57079632679 0.52"/>
 				<geometry>
 					<!-- <mesh filename="package://robotiq_s_model_visualization/meshes/s-model_articulated/collision/link_3.STL" /> -->
-					<box size="0.15 0.03 0.03" />
+					<mesh filename="package://robotiq_s_model_visualization/meshes/s-model_articulated/visual/extensions.STL" />
+					<!-- <box size="0.15 0.03 0.03" /> -->
 				</geometry>
 				<material name="yellow"/>
@@ -153,5 +155,5 @@
 			<parent link="${prefix}link_3"/>
 			<child link="${prefix}link_3_tip"/>
-			<origin xyz="0.15 0.09 0" rpy="0 0 0"/>
+			<origin xyz="0.12 0.06 0" rpy="0 0 0"/>
 		</joint>
 		<!-- end of joint list -->

Commit message: Updated finger tips

File: robotiq_s_model_visualization/cfg/s-model_finger_articulated_macro.xacro (robot description, xacro)
@@ -109,5 +109,5 @@
 				<origin xyz="0 0 0" rpy="0 0 0.52"/>
 				<geometry>
-					<mesh filename="package://robotiq_s_model_visualization/meshes/s-model_articulated/visual/link_3.STL" />
+					<mesh filename="package://robotiq_s_model_visualization/meshes/s-model_articulated/visual/fingers.STL" />
 				</geometry>
 				<material name="green"/>
@@ -116,5 +116,5 @@
 				<origin xyz="0 0 0" rpy="0 0 0.52"/>
 				<geometry>
-					<mesh filename="package://robotiq_s_model_visualization/meshes/s-model_articulated/collision/link_3.STL" />
+					<mesh filename="package://robotiq_s_model_visualization/meshes/s-model_articulated/collision/fingers.STL" />
 				</geometry>
 				<material name="yellow"/>

Commit message: Fixed finger tips

File: robotiq_s_model_visualization/cfg/s-model_finger_articulated_macro.xacro (robot description, xacro)
@@ -107,5 +107,5 @@
 		<link name="${prefix}link_3_tip">
 			<visual>
-				<origin xyz="0 0 0" rpy="0 0 0.52"/>
+				<origin xyz="0 0.01 -0.015" rpy="1.57079632679 0 0.52"/>
 				<geometry>
 					<mesh filename="package://robotiq_s_model_visualization/meshes/s-model_articulated/visual/fingers.STL" />
@@ -116,5 +116,5 @@
 				<origin xyz="0 0 0" rpy="0 0 0.52"/>
 				<geometry>
-					<mesh filename="package://robotiq_s_model_visualization/meshes/s-model_articulated/collision/fingers.STL" />
+					<mesh filename="package://robotiq_s_model_visualization/meshes/s-model_articulated/visual/fingers.STL" />
 				</geometry>
 				<material name="yellow"/>

Commit message: Fixed finger tip orientation

File: robotiq_s_model_visualization/cfg/s-model_finger_articulated_macro.xacro (robot description, xacro)
@@ -114,5 +114,5 @@
 			</visual>
 			<collision>
-				<origin xyz="0 0 0" rpy="0 0 0.52"/>
+				<origin xyz="0 0.01 -0.015" rpy="1.57079632679 0 0.52"/>
 				<geometry>
 					<mesh filename="package://robotiq_s_model_visualization/meshes/s-model_articulated/visual/fingers.STL" />
